File: PentaBlinkyCR2032.brd (EAGLE design)
At the start: 33 x 38.1 mm, 15 parts, among them J1 AVR_SPI_PRG_6LABELED

Commit message: 4H Branding
Parts:
- removed U$3: USER_HACKABLE, logo:USER_HACKABLE
- added U$4: 4H-LOGO6, 4h:4H_LOGO_6
Other:
- board text added: "18 USC 707"
- board text added: "Cache Makers cachemakers.org"
Changed lines of the file:
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@@
 <layer number="20" name="Dimension" color="15" fill="1" visible="yes" active="yes"/>
 <layer number="21" name="tPlace" color="7" fill="1" visible="yes" active="yes"/>
-<layer number="22" name="bPlace" color="7" fill="1" visible="yes" active="yes"/>
+<layer number="22" name="bPlace" color="6" fill="1" visible="yes" active="yes"/>
 <layer number="23" name="tOrigins" color="15" fill="1" visible="yes" active="yes"/>
-<layer number="24" name="bOrigins" color="15" fill="1" visible="yes" active="yes"/>
+<layer number="24" name="bOrigins" color="14" fill="1" visible="yes" active="yes"/>
 <layer number="25" name="tNames" color="7" fill="1" visible="yes" active="yes"/>
-<layer number="26" name="bNames" color="7" fill="1" visible="yes" active="yes"/>
+<layer number="26" name="bNames" color="6" fill="1" visible="yes" active="yes"/>
 <layer number="27" name="tValues" color="7" fill="1" visible="yes" active="yes"/>
-<layer number="28" name="bValues" color="7" fill="1" visible="yes" active="yes"/>
+<layer number="28" name="bValues" color="6" fill="1" visible="yes" active="yes"/>
 <layer number="29" name="tStop" color="7" fill="3" visible="no" active="yes"/>
 <layer number="30" name="bStop" color="7" fill="6" visible="no" active="yes"/>
@@
 <wire x1="3.81" y1="0" x2="29.21" y2="0" width="0" layer="20"/>
 <wire x1="29.21" y1="0" x2="33.02" y2="3.81" width="0" layer="20" curve="90"/>
-<hole x="3.81" y="34.29" drill="3.175"/>
-<hole x="29.21" y="34.29" drill="3.175"/>
+<hole x="3.81" y="34.29" drill="3.81"/>
+<hole x="29.21" y="34.29" drill="3.81"/>
 <text x="26.67" y="8.89" size="1.016" layer="21" align="center">1</text>
 <text x="26.67" y="11.43" size="1.016" layer="21" align="center">2</text>
@@
 <text x="13.335" y="6.35" size="1.016" layer="21" align="center">4</text>
 <text x="6.985" y="6.35" size="1.016" layer="21" align="center">5</text>
-<text x="16.51" y="19.685" size="1.016" layer="21" align="center">User Hackable
+<text x="30.7975" y="27.94" size="0.6096" layer="21" rot="R90" align="center">User Hackable
 Pente Blinky</text>
 <text x="6.35" y="20.32" size="1.016" layer="21" align="center">MODE</text>
@@
 <text x="4.7625" y="14.9225" size="0.8128" layer="22" rot="MR270" align="center">userhackable.com/penteblinky</text>
 <text x="16.51" y="18.0975" size="1.016" layer="22" rot="MR0" align="center">CR2032</text>
+<text x="22.86" y="22.86" size="0.6096" layer="21" rot="R50" align="top-center">18 USC 707</text>
+<text x="1.27" y="25.7175" size="0.8128" layer="21" rot="R90" align="top-center">Cache Makers
+cachemakers.org</text>
 </plain>
 <attributes>
@@
 <attribute name="VALUE" x="20.828" y="22.86" size="1.6764" layer="28" font="vector" rot="MR0"/>
 </element>
-<element name="U$3" library="logo" package="USER_HACKABLE" value="USER_HACKABLE" x="16.51" y="29.21"/>
+<element name="U$4" library="4h" package="4H_LOGO_6" value="4H-LOGO6" x="16.51" y="27.94"/>
 </elements>
 <signals>

Commit message: branding for 4h
Parts:
- U$4: value 4H-LOGO6 -> (none)
Changed lines of the file:
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@@
 </class>
 </classes>
-<designrules name="default">
+<designrules name="LaenPCBOrder">
 <description language="de">&lt;b&gt;EAGLE Design Rules&lt;/b&gt;
 &lt;p&gt;
@@
 Einstellungen hier und speichern die Design Rules unter
 einem neuen Namen ab.</description>
-<description language="en">&lt;b&gt;EAGLE Design Rules&lt;/b&gt;
+<description language="en">&lt;b&gt;Laen's PCB Order Design Rules&lt;/b&gt;
 &lt;p&gt;
-The default Design Rules have been set to cover
-a wide range of applications. Your particular design
-may have different requirements, so please make the
-necessary adjustments and save your customized
-design rules under a new name.</description>
+Please make sure your boards conform to these design rules.</description>
 <param name="layerSetup" value="(1*16)"/>
-<param name="mtCopper" value="0.035mm 0.035mm 0.035mm 0.035mm 0.035mm 0.035mm 0.035mm 0.035mm 0.035mm 0.035mm 0.035mm 0.035mm 0.035mm 0.035mm 0.035mm 0.035mm"/>
-<param name="mtIsolate" value="1.5mm 0.15mm 0.2mm 0.15mm 0.2mm 0.15mm 0.2mm 0.15mm 0.2mm 0.15mm 0.2mm 0.15mm 0.2mm 0.15mm 0.2mm"/>
-<param name="mdWireWire" value="8mil"/>
-<param name="mdWirePad" value="8mil"/>
-<param name="mdWireVia" value="8mil"/>
-<param name="mdPadPad" value="8mil"/>
-<param name="mdPadVia" value="8mil"/>
-<param name="mdViaVia" value="8mil"/>
-<param name="mdSmdPad" value="8mil"/>
-<param name="mdSmdVia" value="8mil"/>
-<param name="mdSmdSmd" value="8mil"/>
+<param name="mtCopper" value="0.0356mm 0.0356mm 0.0356mm 0.0356mm 0.0356mm 0.0356mm 0.0356mm 0.0356mm 0.0356mm 0.0356mm 0.0356mm 0.0356mm 0.0356mm 0.0356mm 0.0356mm 0.0356mm"/>
+<param name="mtIsolate" value="1.5011mm 0.1499mm 0.2007mm 0.1499mm 0.2007mm 0.1499mm 0.2007mm 0.1499mm 0.2007mm 0.1499mm 0.2007mm 0.1499mm 0.2007mm 0.1499mm 0.2007mm"/>
+<param name="mdWireWire" value="6mil"/>
+<param name="mdWirePad" value="6mil"/>
+<param name="mdWireVia" value="6mil"/>
+<param name="mdPadPad" value="6mil"/>
+<param name="mdPadVia" value="6mil"/>
+<param name="mdViaVia" value="6mil"/>
+<param name="mdSmdPad" value="6mil"/>
+<param name="mdSmdVia" value="6mil"/>
+<param name="mdSmdSmd" value="6mil"/>
 <param name="mdViaViaSameLayer" value="8mil"/>
 <param name="mnLayersViaInSmd" value="2"/>
-<param name="mdCopperDimension" value="40mil"/>
-<param name="mdDrill" value="8mil"/>
+<param name="mdCopperDimension" value="15mil"/>
+<param name="mdDrill" value="6mil"/>
 <param name="mdSmdStop" value="0mil"/>
-<param name="msWidth" value="10mil"/>
-<param name="msDrill" value="24mil"/>
-<param name="msMicroVia" value="9.99mm"/>
+<param name="msWidth" value="6mil"/>
+<param name="msDrill" value="13mil"/>
+<param name="msMicroVia" value="13mil"/>
 <param name="msBlindViaRatio" value="0.5"/>
 <param name="rvPadTop" value="0.25"/>
@@
 <param name="rvMicroViaOuter" value="0.25"/>
 <param name="rvMicroViaInner" value="0.25"/>
-<param name="rlMinPadTop" value="10mil"/>
+<param name="rlMinPadTop" value="7mil"/>
 <param name="rlMaxPadTop" value="20mil"/>
-<param name="rlMinPadInner" value="10mil"/>
+<param name="rlMinPadInner" value="7mil"/>
 <param name="rlMaxPadInner" value="20mil"/>
-<param name="rlMinPadBottom" value="10mil"/>
+<param name="rlMinPadBottom" value="7mil"/>
 <param name="rlMaxPadBottom" value="20mil"/>
-<param name="rlMinViaOuter" value="8mil"/>
+<param name="rlMinViaOuter" value="7mil"/>
 <param name="rlMaxViaOuter" value="20mil"/>
-<param name="rlMinViaInner" value="8mil"/>
+<param name="rlMinViaInner" value="7mil"/>
 <param name="rlMaxViaInner" value="20mil"/>
 <param name="rlMinMicroViaOuter" value="4mil"/>
@@
 <param name="mvStopFrame" value="1"/>
 <param name="mvCreamFrame" value="0"/>
-<param name="mlMinStopFrame" value="4mil"/>
-<param name="mlMaxStopFrame" value="4mil"/>
+<param name="mlMinStopFrame" value="3mil"/>
+<param name="mlMaxStopFrame" value="3mil"/>
 <param name="mlMinCreamFrame" value="0mil"/>
 <param name="mlMaxCreamFrame" value="0mil"/>
@@
 <attribute name="VALUE" x="20.828" y="22.86" size="1.6764" layer="28" font="vector" rot="MR0"/>
 </element>
-<element name="U$4" library="4h" package="4H_LOGO_6" value="4H-LOGO6" x="16.51" y="27.94"/>
+<element name="U$4" library="4h" package="4H_LOGO_6" value="" x="16.51" y="27.94"/>
 </elements>
 <signals>
